File: Hardware/SparkFun_IoT_RedBoard-RP2350.kicad_pcb (KiCad board)
At the start: 4 copper layers, 68.6 x 58.4 mm, 236 parts, among them J1 Conn_01x08_SMD_Combined, J10 Conn_01x03, J11 Conn_01x22_FPC_0.5mm_HSTX_Ver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, J12 Qwiic_RA, J13 microSD, J14 JST_1mm_3_Vertical, J2 Conn_01x06_SMD_Combined, J3 Barrel_Jack_SMD, J4 USB_C_Receptacle, J5 Conn_01x04_SolderPads, J6 Conn_01x02, J7 JST_2mm_LiPo, J8 Conn_01x10_SMD_Combined, J9 Conn_01x08_SMD_Combined, Q1 RE1C001ZPTL, SW1 BOOT, SW2 RESET, SW3 USER, U1 RP2350B, U10 RT9080-3.3, U2 RM2, U3 W25Q128JVPIM, U4 APS6404L-3SQR-ZR, U5 LM66200, U6 AP63357DV-7, U7 LM66200, U8 MAX17048, U9 MCP73831, Y1 12MHz

Commit message: Update v01 from checklist. Added measures.
Parts:
- removed kibuzzard-676083F1: G***, kibuzzard-676083F1
- removed kibuzzard-67608407: G***, kibuzzard-67608407
- removed kibuzzard-6760842C: G***, kibuzzard-6760842C
- added kibuzzard-6761DE7B: G***, kibuzzard-6761DE7B, F.Cu at (140.4, 82.0)
- added kibuzzard-6761DE89: G***, kibuzzard-6761DE89, F.Cu at (130.8, 82.0)
- added kibuzzard-6761DE91: G***, kibuzzard-6761DE91, F.Cu at (124.6, 75.0)
- added kibuzzard-6761DF2F: G***, kibuzzard-6761DF2F, F.Cu at (142.0, 74.5)
- added kibuzzard-6761DF7C: G***, kibuzzard-6761DF7C, F.Cu at (139.5, 74.8)
- JP1: value ~ -> SHLD
- JP6: value ~ -> PWR
- U2: footprint SparkFun_XRP_Controller:RM2_Tight -> SparkFun-RF:RM2_Tight
- moved C7 0.20 mm to (162.6, 92.5)
- renumbered C26 to C25, C25 to C26, J14 to J12, J12 to J13, J13 to J14, R31 to R11, R32 to R12, R11 to R13, R12 to R14, R13 to R15, R14 to R16, R15 to R17, R16 to R18, R17 to R19, R18 to R20, R19 to R21, R20 to R22, R21 to R23, R22 to R24, R23 to R25, R24 to R26, R25 to R27, R26 to R28, R27 to R29, R28 to R30, R29 to R31, R30 to R32, TP3 to TP1, TP12 to TP10, TP13 to TP11, TP4 to TP2, TP5 to TP3, TP6 to TP4, TP7 to TP5, TP8 to TP6, TP9 to TP7, TP10 to TP8, TP11 to TP9
Routing:
- net GND: track 43.0 -> 44.1 mm, vias 199 -> 198
- net 1.1V: track 36.8 -> 37.5 mm
- net /Core/~{STAT}: track 28.6 -> 28.2 mm, vias 3 -> 2
- net 3.3V: vias 33 -> 31
- net /Core/WRL_IO0: vias 3 -> 2
Other:
- board text added: "Finish: Lead-Free HASL"
- board text removed: "Finish: ENIG"
