File: Hardware/SparkFun_IoT_RedBoard-RP2350.kicad_pcb (KiCad board)
At the start: 4 copper layers, 68.6 x 58.4 mm, 238 parts, among them J1 Conn_01x08_SMD_Combined, J10 Conn_01x03, J11 Conn_01x22_FPC_0.5mm_HSTX_Ver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, J12 JST_1mm_3_Vertical, J13 Qwiic_RA, J14 microSD, J2 Conn_01x06_SMD_Combined, J3 Barrel_Jack_SMD, J4 USB_C_Receptacle, J5 Conn_01x04_SolderPads, J6 Conn_01x02, J7 JST_2mm_LiPo, J8 Conn_01x10_SMD_Combined, J9 Conn_01x08_SMD_Combined, Q1 RE1C001ZPTL, SW1 BOOT, SW2 RESET, SW3 USER, U1 RP2350B, U10 RT9080-3.3, U2 RM2, U3 W25Q128JVPIM, U4 APS6404L-3SQR-ZR, U5 LM66200, U6 AP63357DV-7, U7 LM66200, U8 MAX17048, U9 MCP73831, Y1 12MHz

Commit message: v01 post design review changes. Panelize/CAM.
Remove F3.
Added switched power for qwiic, rgb, sd.
Update USB diode for prod friendly package.
Added debounce cap on User button.
Swap user and boot buttons.
Make F2 a smaller package.
Renumber GPIO and use contiguous numbers for PIO purposes.
Swap inputs on Ideal diodes for battery powered current purposes.
Move USB termination resistors closer to MCU.
Fixed A0-A5 ordering.
Update silks.
Add mask to middle of SMD GPIOs.
Parts:
- removed the C25 at (153.9, 109.2)
- removed F3: 6V/2.0A/4.0A, SparkFun-Fuse:1210
- removed kibuzzard-6757671D: G***, kibuzzard-6757671D
- removed kibuzzard-676089E6: G***, kibuzzard-676089E6
- removed kibuzzard-67608C2D: G***, kibuzzard-67608C2D
- removed kibuzzard-67608C3D: G***, kibuzzard-67608C3D
- removed kibuzzard-67608C4F: G***, kibuzzard-67608C4F
- removed kibuzzard-67608F6B: G***, kibuzzard-67608F6B
- removed kibuzzard-676090AD: G***, kibuzzard-676090AD
- removed kibuzzard-67609282: G***, kibuzzard-67609282
- removed kibuzzard-67609463: G***, kibuzzard-67609463
- removed kibuzzard-6760946E: G***, kibuzzard-6760946E
- removed kibuzzard-6760947A: G***, kibuzzard-6760947A
- removed kibuzzard-6761DE7B: G***, kibuzzard-6761DE7B
- added C26: 0.1uF, SparkFun-Capacitor:C_0402_1005Metric, F.Cu at (132.0, 114.5)
- added C30: 2.2uF, SparkFun-Capacitor:C_0402_1005Metric, F.Cu at (152.6, 108.6)
- added C31: 2.2uF, SparkFun-Capacitor:C_0402_1005Metric, F.Cu at (150.4, 108.6)
- added C36: 0.1uF, SparkFun-Capacitor:C_0402_1005Metric, F.Cu at (126.0, 79.9)
- added R24: 10k, SparkFun-Resistor:R_0402_1005Metric, F.Cu at (154.7, 105.6)
- added R25: 1M, SparkFun-Resistor:R_0402_1005Metric, F.Cu at (154.7, 106.7)
- added R33: 10k, SparkFun-Resistor:R_0402_1005Metric, F.Cu at (132.1, 91.0)
- added U10: RT9080-3.3, SparkFun-Semiconductor-Standard:SOT23-5, F.Cu at (151.5, 106.2)
- added kibuzzard-67643BB7: G***, kibuzzard-67643BB7, F.Cu at (130.8, 82.0)
- added kibuzzard-67658D2A: G***, kibuzzard-67658D2A, F.Cu at (120.6, 119.3)
- added kibuzzard-6765AF34: G***, kibuzzard-6765AF34, F.Cu at (146.1, 115.4)
- added kibuzzard-6765AF51: G***, kibuzzard-6765AF51, F.Cu at (143.5, 114.8)
- added kibuzzard-6765B0D7: G***, kibuzzard-6765B0D7, B.Cu at (149.3, 106.2)
- added kibuzzard-6765B610: G***, kibuzzard-6765B610, F.Cu at (154.7, 74.9)
- added kibuzzard-6765B61A: G***, kibuzzard-6765B61A, F.Cu at (157.2, 74.9)
- added kibuzzard-6765B620: G***, kibuzzard-6765B620, F.Cu at (161.3, 74.9)
- added kibuzzard-6765B634: G***, kibuzzard-6765B634, B.Cu at (161.3, 69.4)
- added kibuzzard-6765B639: G***, kibuzzard-6765B639, B.Cu at (157.2, 69.5)
- added kibuzzard-6765B63E: G***, kibuzzard-6765B63E, B.Cu at (154.7, 69.5)
- added kibuzzard-6765B674: G***, kibuzzard-6765B674, F.Cu at (164.7, 108.5)
- added kibuzzard-6765D4E3: G***, kibuzzard-6765D4E3, F.Cu at (153.7, 115.9)
- added kibuzzard-6765D50A: G***, kibuzzard-6765D50A, F.Cu at (151.1, 115.4)
- added kibuzzard-6765D50A: G***, kibuzzard-6765D50A, B.Cu at (151.2, 120.7)
- D2: value PRTR5V0U2F -> DT1042-04SO; footprint Package_TO_SOT_SMD:SOT-886 -> SparkFun-Semiconductor-Standard:SOT23-6
- F2: value 6V/2.0A/4.0A -> 6V/0.75A/1.5A; footprint SparkFun-Fuse:1210 -> SparkFun-Fuse:1206
- JP4: moved to B.Cu
- JP5: value BUS -> LP; footprint SparkFun-Jumper:Jumper_2_NO -> SparkFun-Jumper:Jumper_2_NC_Trace
- moved kibuzzard-67608CF1 12.7 mm to (166.4, 115.6)
- moved kibuzzard-6760916E 12.7 mm to (166.4, 120.0)
- moved kibuzzard-676091D0 12.7 mm to (179.1, 119.9)
- moved kibuzzard-67608E02 12.7 mm to (179.1, 115.5)
- moved R4 12.3 mm to (139.3, 83.3)
- moved R3 12.3 mm to (139.3, 84.5)
- moved Ref** 10.5 mm to (119.1, 121.7)
- moved TP11 10.2 mm to (130.8, 78.7)
- moved TP9 10.2 mm to (141.0, 78.7)
- moved SW1 9.60 mm to (140.4, 78.5)
- moved SW3 9.60 mm to (130.8, 78.5)
- moved kibuzzard-6761DE89 9.60 mm to (140.4, 82.0)
- moved R35 9.50 mm to (135.6, 79.9)
- moved R9 9.50 mm to (145.1, 79.9)
- moved kibuzzard-676084E8 7.73 mm to (127.7, 122.9)
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- renumbered C26 to C25, C30 to C32, C31 to C33, C32 to C34, C33 to C35, R24 to R22, R22 to R23, R23 to R26, R25 to R27, R26 to R28, R27 to R29, R28 to R30, R29 to R31, R30 to R32, R31 to R34, R32 to R35, U10 to U11, U6 to U5, U5 to U6
Connections:
- net /Core/~{BATT_PWR} renamed /Core/BATT_PWR
- C34 pad 1: 3.3V -> 3.3V_P
- C35 pad 1: 3.3V -> 3.3V_P
- D2 pad 4: /UD+ -> /USBC+
- D2 pad 6: /UD- -> /USBC-
- D4 pad 4: 3.3V -> 3.3V_P
- H1 pad D7: /IO37 -> /IO33
- H1 pad D8: /IO38 -> /IO34
- H1 pad D9: /IO39 -> /IO35
- J13 pad 2: 3.3V -> 3.3V_P
- J14 pad 4: 3.3V -> 3.3V_P
- J2 pad 1: /A0 -> /A5
- J2 pad 2: /A1 -> /A4
- J2 pad 3: /A2 -> /A3
- J2 pad 4: /A3 -> /A2
- J2 pad 5: /A4 -> /A1
- J2 pad 6: /A5 -> /A0
- J3 pad GNDBREAK: /Core/~{BARREL} -> unconnected-(J3-PadGNDBREAK)
- J5 pad 2: /USBC+ -> /USBC-
- J5 pad 3: /USBC- -> /USBC+
- J8 pad 10: /IO38 -> /IO34
- J8 pad 9: /IO39 -> /IO35
- J9 pad 1: /IO37 -> /IO33
- JP3 pad 2: 3.3V -> 3.3V_P
- JP4 pad 2: Net-(JP4-B) -> VBUS
- JP5 pad 1: Net-(JP4-B) -> 3.3V
- JP5 pad 2: VBUS -> Net-(JP5-B)
- R3 pad 1: /UD+ -> /USBC+
- R4 pad 1: /UD- -> /USBC-
- U1 pad 4: /Core/~{BARREL} -> /Core/PERI_POW
- U1 pad 42: /Core/WRL_~{CS} -> /IO33
- U1 pad 43: /Core/WRL_CLK -> /IO34
- U1 pad 44: /Core/WRL_DAT -> /IO35
- U1 pad 45: /Core/~{USER_BTN} -> /Core/WRL_~{CS}
- U1 pad 46: /IO37 -> /Core/WRL_CLK
- U1 pad 47: /IO38 -> /Core/WRL_DAT
- U1 pad 48: /IO39 -> /Core/~{USER_BTN}
- U6 pad 3: VUSB -> VDD
- U6 pad 6: VDD -> VUSB
- U7 pad 3: 5V -> VBATT
- U7 pad 6: VBATT -> 5V
Routing:
- net 3.3V_P: track 0.00 -> 115.4 mm, vias 0 -> 6
- net /Core/~{BARREL}: track 44.9 -> 0.00 mm, vias 4 -> 0
- net /Core/PERI_POW: track 0.00 -> 19.9 mm, vias 0 -> 4
- net /IO33: track 0.00 -> 19.1 mm
- net /IO37: track 18.8 -> 0.00 mm
- net /IO34: track 0.00 -> 15.5 mm
- net /USBC+: track 9.47 -> 24.9 mm
- net /IO38: track 15.2 -> 0.00 mm
- net /IO35: track 0.00 -> 15.0 mm
- net /IO39: track 14.5 -> 0.00 mm, vias 2 -> 0
- net /USBC-: track 10.6 -> 23.4 mm
- net /Core/USB.D-: track 22.5 -> 9.73 mm
- net /Core/USB.D+: track 22.5 -> 9.73 mm
- net /Core/FLASH_~{CS}: track 35.5 -> 42.5 mm
- net /Core/~{USER_BTN}: track 29.2 -> 36.0 mm, vias 3 -> 1
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- removed copper zone on F.Cu, net Net-(JP4-B)

Commit message: Update for reds
Change version number to v10.
Make user button number correct.
Rotate HSTX conn 180 degrees electrically.
Add silk for HSTX contact direction.
Increase silk text size where it made sense.
Increase silk label length on PTHs.
Panelize and CAM.
Parts:
- removed kibuzzard-67607EA7: G***, kibuzzard-67607EA7
- removed kibuzzard-67608548 (x2): G***, kibuzzard-67608548
- removed kibuzzard-67608565 (x2): G***, kibuzzard-67608565
- removed kibuzzard-67608870: G***, kibuzzard-67608870
- removed kibuzzard-6760893C: G***, kibuzzard-6760893C
- removed kibuzzard-67608B72: G***, kibuzzard-67608B72
- removed kibuzzard-67608B85: G***, kibuzzard-67608B85
- removed kibuzzard-67608BA5: G***, kibuzzard-67608BA5
- removed kibuzzard-67608BC2: G***, kibuzzard-67608BC2
- removed kibuzzard-67608BDC: G***, kibuzzard-67608BDC
- removed kibuzzard-67608BED: G***, kibuzzard-67608BED
- removed kibuzzard-67608C5B: G***, kibuzzard-67608C5B
- removed kibuzzard-67608C6C: G***, kibuzzard-67608C6C
- removed kibuzzard-67608C7C: G***, kibuzzard-67608C7C
- removed kibuzzard-67608C9A: G***, kibuzzard-67608C9A
- removed kibuzzard-67608CA9: G***, kibuzzard-67608CA9
- removed kibuzzard-67608CBD: G***, kibuzzard-67608CBD
- removed kibuzzard-67608CCA: G***, kibuzzard-67608CCA
- removed kibuzzard-67608CF1: G***, kibuzzard-67608CF1
- removed kibuzzard-67608CFE: G***, kibuzzard-67608CFE
- removed kibuzzard-67608D10: G***, kibuzzard-67608D10
- removed kibuzzard-67608D56: G***, kibuzzard-67608D56
- removed kibuzzard-67608DF4: G***, kibuzzard-67608DF4
- removed kibuzzard-67608E02: G***, kibuzzard-67608E02
- removed kibuzzard-67609166: G***, kibuzzard-67609166
- removed kibuzzard-6760916E: G***, kibuzzard-6760916E
- removed kibuzzard-6760917F: G***, kibuzzard-6760917F
- removed kibuzzard-6760919A: G***, kibuzzard-6760919A
- removed kibuzzard-676091AE: G***, kibuzzard-676091AE
- removed kibuzzard-676091D0: G***, kibuzzard-676091D0
- removed kibuzzard-6760921E: G***, kibuzzard-6760921E
- removed kibuzzard-67609232 (x4): G***, kibuzzard-67609232
- removed kibuzzard-6760926E: G***, kibuzzard-6760926E
- removed kibuzzard-676092A4: G***, kibuzzard-676092A4
- removed kibuzzard-676092CD: G***, kibuzzard-676092CD
- removed kibuzzard-6760931F: G***, kibuzzard-6760931F
- removed kibuzzard-6760934B: G***, kibuzzard-6760934B
- removed kibuzzard-67609371: G***, kibuzzard-67609371
- removed kibuzzard-6760941C: G***, kibuzzard-6760941C
- removed kibuzzard-67609429: G***, kibuzzard-67609429
- removed kibuzzard-67609439: G***, kibuzzard-67609439
- removed kibuzzard-6760944A: G***, kibuzzard-6760944A
- removed kibuzzard-67609456: G***, kibuzzard-67609456
- removed kibuzzard-676094B8: G***, kibuzzard-676094B8
- removed kibuzzard-676094CB: G***, kibuzzard-676094CB
- removed kibuzzard-676094D3: G***, kibuzzard-676094D3
- removed kibuzzard-67609507: G***, kibuzzard-67609507
- removed kibuzzard-6760951B: G***, kibuzzard-6760951B
- removed kibuzzard-67609537: G***, kibuzzard-67609537
- removed kibuzzard-6760955F: G***, kibuzzard-6760955F
- removed kibuzzard-67609575: G***, kibuzzard-67609575
- removed kibuzzard-67609587: G***, kibuzzard-67609587
- removed kibuzzard-6760981A: G***, kibuzzard-6760981A
- removed kibuzzard-67609A17: G***, kibuzzard-67609A17
- removed kibuzzard-67609A8A: G***, kibuzzard-67609A8A
- removed kibuzzard-6761DF2F: G***, kibuzzard-6761DF2F
- removed kibuzzard-6761DF7C: G***, kibuzzard-6761DF7C
- removed kibuzzard-67643BB7: G***, kibuzzard-67643BB7
- removed kibuzzard-67658D2A: G***, kibuzzard-67658D2A
- removed kibuzzard-6765B0D7: G***, kibuzzard-6765B0D7
- removed kibuzzard-6765B610: G***, kibuzzard-6765B610
- removed kibuzzard-6765B61A: G***, kibuzzard-6765B61A
- removed kibuzzard-6765B620: G***, kibuzzard-6765B620
- removed kibuzzard-6765B634: G***, kibuzzard-6765B634
- removed kibuzzard-6765B639: G***, kibuzzard-6765B639
- removed kibuzzard-6765B63E: G***, kibuzzard-6765B63E
- removed kibuzzard-6765D4E3: G***, kibuzzard-6765D4E3
- removed kibuzzard-6765D50A (x2): G***, kibuzzard-6765D50A
- added kibuzzard-67A3E09E: G***, kibuzzard-67A3E09E, F.Cu at (179.1, 85.3)
- added kibuzzard-67A3E0D1: G***, kibuzzard-67A3E0D1, F.Cu at (179.1, 74.2)
- added kibuzzard-67A3E112: G***, kibuzzard-67A3E112, F.Cu at (176.6, 74.2)
- added kibuzzard-67A3E12A: G***, kibuzzard-67A3E12A, F.Cu at (174.0, 74.5)
- added kibuzzard-67A3E140: G***, kibuzzard-67A3E140, F.Cu at (171.5, 74.5)
- added kibuzzard-67A3E168: G***, kibuzzard-67A3E168, F.Cu at (169.0, 74.5)
- added kibuzzard-67A3E171: G***, kibuzzard-67A3E171, F.Cu at (166.4, 74.5)
- added kibuzzard-67A3E17B: G***, kibuzzard-67A3E17B, F.Cu at (163.9, 74.5)
- added kibuzzard-67A3E183: G***, kibuzzard-67A3E183, F.Cu at (161.3, 74.5)
- added kibuzzard-67A3E1A1: G***, kibuzzard-67A3E1A1, F.Cu at (157.2, 74.5)
- added kibuzzard-67A3E1A7: G***, kibuzzard-67A3E1A7, F.Cu at (154.7, 74.5)
- added kibuzzard-67A3E1AE: G***, kibuzzard-67A3E1AE, F.Cu at (152.2, 74.5)
- added kibuzzard-67A3E1B5: G***, kibuzzard-67A3E1B5, F.Cu at (149.6, 74.5)
- added kibuzzard-67A3E1BE: G***, kibuzzard-67A3E1BE, F.Cu at (147.1, 74.5)
- added kibuzzard-67A3E1C5: G***, kibuzzard-67A3E1C5, F.Cu at (144.5, 74.5)
- added kibuzzard-67A3E1CD: G***, kibuzzard-67A3E1CD, F.Cu at (142.0, 74.0)
- added kibuzzard-67A3E1E0: G***, kibuzzard-67A3E1E0, F.Cu at (139.5, 74.4)
- added kibuzzard-67A3E1FA: G***, kibuzzard-67A3E1FA, F.Cu at (136.9, 74.2)
- added kibuzzard-67A3E201: G***, kibuzzard-67A3E201, F.Cu at (134.4, 74.2)
- added kibuzzard-67A3E20D: G***, kibuzzard-67A3E20D, F.Cu at (130.8, 82.0)
- added kibuzzard-67A3E235: G***, kibuzzard-67A3E235, F.Cu at (179.1, 116.0)
- added kibuzzard-67A3E24D: G***, kibuzzard-67A3E24D, F.Cu at (176.5, 116.0)
- added kibuzzard-67A3E254: G***, kibuzzard-67A3E254, F.Cu at (174.1, 116.0)
- added kibuzzard-67A3E25A: G***, kibuzzard-67A3E25A, F.Cu at (171.5, 116.0)
- added kibuzzard-67A3E263: G***, kibuzzard-67A3E263, F.Cu at (169.0, 116.0)
- added kibuzzard-67A3E26A: G***, kibuzzard-67A3E26A, F.Cu at (166.4, 116.0)
- added kibuzzard-67A3E284: G***, kibuzzard-67A3E284, F.Cu at (153.7, 116.2)
- added kibuzzard-67A3E2A5: G***, kibuzzard-67A3E2A5, F.Cu at (151.1, 115.9)
- added kibuzzard-67A3E2C6: G***, kibuzzard-67A3E2C6, F.Cu at (148.6, 115.7)
- added kibuzzard-67A3E41E: G***, kibuzzard-67A3E41E, B.Cu at (124.6, 113.3)
- added kibuzzard-67A3E43C: G***, kibuzzard-67A3E43C, B.Cu at (132.7, 112.4)
- added kibuzzard-67A3E455: G***, kibuzzard-67A3E455, B.Cu at (135.9, 111.5)
- added kibuzzard-67A3E45D: G***, kibuzzard-67A3E45D, B.Cu at (138.5, 111.5)
- added kibuzzard-67A3E4A3: G***, kibuzzard-67A3E4A3, B.Cu at (149.2, 106.2)
- added kibuzzard-67A3E4D1: G***, kibuzzard-67A3E4D1, B.Cu at (165.6, 110.5)
- added kibuzzard-67A3F3F2: G***, kibuzzard-67A3F3F2, B.Cu at (153.8, 114.5)
- added kibuzzard-67A3F4AA: G***, kibuzzard-67A3F4AA, B.Cu at (120.9, 89.0)
- added kibuzzard-67A3F4E6: G***, kibuzzard-67A3F4E6, B.Cu at (134.4, 70.7)
- added kibuzzard-67A3F532: G***, kibuzzard-67A3F532, B.Cu at (136.9, 70.7)
- added kibuzzard-67A3F552: G***, kibuzzard-67A3F552, B.Cu at (139.5, 70.1)
- added kibuzzard-67A3F565: G***, kibuzzard-67A3F565, B.Cu at (142.0, 69.7)
- added kibuzzard-67A3F577: G***, kibuzzard-67A3F577, B.Cu at (144.5, 70.9)
- added kibuzzard-67A3F59C: G***, kibuzzard-67A3F59C, B.Cu at (147.1, 71.1)
- added kibuzzard-67A3F5C2: G***, kibuzzard-67A3F5C2, B.Cu at (149.6, 71.1)
- added kibuzzard-67A3F5D5: G***, kibuzzard-67A3F5D5, B.Cu at (152.2, 70.3)
- added kibuzzard-67A3F5FB: G***, kibuzzard-67A3F5FB, B.Cu at (154.7, 69.4)
- added kibuzzard-67A3F625: G***, kibuzzard-67A3F625, B.Cu at (157.2, 69.4)
- added kibuzzard-67A3F62C: G***, kibuzzard-67A3F62C, B.Cu at (161.3, 69.4)
- added kibuzzard-67A3F633: G***, kibuzzard-67A3F633, B.Cu at (163.8, 69.4)
- added kibuzzard-67A3F639: G***, kibuzzard-67A3F639, B.Cu at (166.4, 69.4)
- added kibuzzard-67A3F63E: G***, kibuzzard-67A3F63E, B.Cu at (168.9, 69.4)
- added kibuzzard-67A3F646: G***, kibuzzard-67A3F646, B.Cu at (171.5, 69.4)
- added kibuzzard-67A3F64D: G***, kibuzzard-67A3F64D, B.Cu at (174.0, 69.4)
- added kibuzzard-67A3F657: G***, kibuzzard-67A3F657, B.Cu at (176.5, 70.6)
- added kibuzzard-67A3F666: G***, kibuzzard-67A3F666, B.Cu at (179.1, 70.4)
- added kibuzzard-67A3F682: G***, kibuzzard-67A3F682, B.Cu at (168.8, 80.4)
- added kibuzzard-67A3F699: G***, kibuzzard-67A3F699, B.Cu at (167.8, 83.0)
- added kibuzzard-67A3F6A9: G***, kibuzzard-67A3F6A9, B.Cu at (169.0, 85.5)
- added kibuzzard-67A3F6CD: G***, kibuzzard-67A3F6CD, B.Cu at (143.5, 119.6)
- added kibuzzard-67A3F6E9: G***, kibuzzard-67A3F6E9, B.Cu at (146.1, 120.1)
- added kibuzzard-67A3F71F: G***, kibuzzard-67A3F71F, B.Cu at (148.6, 119.9)
- added kibuzzard-67A3F72C: G***, kibuzzard-67A3F72C, B.Cu at (151.2, 121.0)
- added kibuzzard-67A3F73E: G***, kibuzzard-67A3F73E, B.Cu at (153.7, 121.4)
- added kibuzzard-67A3F74E: G***, kibuzzard-67A3F74E, B.Cu at (156.2, 120.9)
- added kibuzzard-67A3F769: G***, kibuzzard-67A3F769, B.Cu at (158.7, 120.9)
- added kibuzzard-67A3F773: G***, kibuzzard-67A3F773, B.Cu at (161.3, 121.1)
- added kibuzzard-67A3F78A: G***, kibuzzard-67A3F78A, B.Cu at (166.4, 120.1)
- added kibuzzard-67A3F799: G***, kibuzzard-67A3F799, B.Cu at (168.9, 120.1)
- added kibuzzard-67A3F7A5: G***, kibuzzard-67A3F7A5, B.Cu at (171.5, 120.1)
- added kibuzzard-67A3F7B2: G***, kibuzzard-67A3F7B2, B.Cu at (174.0, 120.1)
- added kibuzzard-67A3F7C3: G***, kibuzzard-67A3F7C3, B.Cu at (176.6, 120.4)
- added kibuzzard-67A3F7D3: G***, kibuzzard-67A3F7D3, B.Cu at (179.1, 120.2)
- added kibuzzard-67A3F996: G***, kibuzzard-67A3F996, F.Cu at (119.2, 121.5)
- added kibuzzard-67A3F9C4: G***, kibuzzard-67A3F9C4, F.Cu at (135.9, 111.0)
- added kibuzzard-67A3F9DC: G***, kibuzzard-67A3F9DC, F.Cu at (138.5, 111.0)
- moved kibuzzard-67608A60 2.20 mm to (121.9, 79.9)
- moved kibuzzard-67608A88 2.15 mm to (121.9, 85.2)
- moved Ref** 1.60 mm to (119.2, 123.3)
- moved kibuzzard-67608AA5 1.60 mm to (121.6, 83.5)
- moved kibuzzard-67608A8F 1.55 mm to (121.6, 81.7)
- moved kibuzzard-676083AD 0.20 mm to (158.9, 104.4) (x2)
- turned J11 to 90 degrees
Connections:
- J11 pad 1: GND -> 3.3V
- J11 pad 11: /Core/IO13_HSTX1 -> /Core/IO12_HSTX0
- J11 pad 12: /Core/IO12_HSTX0 -> /Core/IO13_HSTX1
- J11 pad 14: unconnected-(J11-Pin_14-Pad14) -> /Core/IO14_HSTX2
- J11 pad 15: unconnected-(J11-Pin_15-Pad15) -> /Core/IO15_HSTX3
- J11 pad 17: /IO29 -> /Core/IO16_HSTX4
- J11 pad 18: /IO28 -> /Core/IO17_HSTX5
- J11 pad 2: /Core/IO19_HSTX7 -> /IO4_SDA
- J11 pad 20: /IO5_SCL -> /Core/IO18_HSTX6
- J11 pad 21: /IO4_SDA -> /Core/IO19_HSTX7
- J11 pad 22: 3.3V -> GND
- J11 pad 3: /Core/IO18_HSTX6 -> /IO5_SCL
- J11 pad 5: /Core/IO17_HSTX5 -> /IO28
- J11 pad 6: /Core/IO16_HSTX4 -> /IO29
- J11 pad 8: /Core/IO15_HSTX3 -> unconnected-(J11-Pin_8-Pad8)
- J11 pad 9: /Core/IO14_HSTX2 -> unconnected-(J11-Pin_9-Pad9)
Other:
- board text added: "v10"
- board text removed: "v01"

Commit message: Update post reds review
Added SOT489
Move vias around so they don't interfere with silk
Change Barrel Jack voltage range.
Increase VUSB trace width.
Add silk to HSTX connector.
Panelize & CAM.
Parts:
- removed kibuzzard-67A3E41E: G***, kibuzzard-67A3E41E
- removed kibuzzard-67A3F996: G***, kibuzzard-67A3F996
- added kibuzzard-67A657F3: G***, kibuzzard-67A657F3, F.Cu at (119.2, 121.5)
- added kibuzzard-67A657FD: G***, kibuzzard-67A657FD, B.Cu at (124.6, 113.3)
- moved kibuzzard-676080F0 1.41 mm to (143.6, 90.6)
- moved G*** 1.35 mm to (151.2, 95.8)
- moved kibuzzard-67608662 1.25 mm to (150.5, 101.7)
- moved kibuzzard-67A3E4D1 1.04 mm to (165.3, 109.5)
- moved G*** 0.40 mm to (152.0, 86.5)
- moved kibuzzard-67608476 0.40 mm to (175.3, 95.0)
- moved C13 0.30 mm to (146.4, 86.1)
- moved C16 0.25 mm to (160.3, 87.8)
- moved R16 0.10 mm to (139.4, 93.8)
Routing:
- net /IO28: track 54.6 -> 53.6 mm
- net /IO5_SCL: track 138.2 -> 139.0 mm
- net /Core/VIN_MEAS: track 41.0 -> 41.7 mm
- net 1.1V: track 37.5 -> 36.8 mm
- net GND: track 39.8 -> 39.2 mm, vias 206 -> 211
