File: Hardware/core.kicad_sch (KiCad schematic)
At the start: 46 parts, among them Q1 RE1C001ZPTL, U1 RP2350B, U2 RM2, U3 W25Q128JVPIM, U4 APS6404L-3SQR-ZR, Y1 12MHz

Commit message: Update v01 from checklist. Added measures.
Parts:
- U2: footprint SparkFun_XRP_Controller:RM2_Tight -> SparkFun-RF:RM2_Tight; symbol SparkFun_XRP_Controller:RM2_Tight -> SparkFun-RF:RM2_Tight
- renumbered R31 to R11, R32 to R12, R11 to R13, R12 to R14, R13 to R15, R14 to R16, R15 to R17, TP3 to TP1, TP4 to TP2, TP5 to TP3, TP6 to TP4, TP7 to TP5, TP8 to TP6, TP9 to TP7

Commit message: v01 post design review changes. Panelize/CAM.
Remove F3.
Added switched power for qwiic, rgb, sd.
Update USB diode for prod friendly package.
Added debounce cap on User button.
Swap user and boot buttons.
Make F2 a smaller package.
Renumber GPIO and use contiguous numbers for PIO purposes.
Swap inputs on Ideal diodes for battery powered current purposes.
Move USB termination resistors closer to MCU.
Fixed A0-A5 ordering.
Update silks.
Add mask to middle of SMD GPIOs.
Connections:
- net IO37 is gone; now on net WRL_CLK: U1.46 (GPIO37)
- net IO38 is gone; now on net WRL_DAT: U1.47 (GPIO38)
- net IO39 is gone; now on net ~{USER_BTN}: U1.48 (GPIO39)
- net WRL_CLK: no longer U1.43 (GPIO34)
- net WRL_DAT: no longer U1.44 (GPIO35)
- net WRL_~{CS}: now also U1.45 (GPIO36); no longer U1.42 (GPIO33)
- net ~{USER_BTN}: no longer U1.45 (GPIO36)
- net ~{BARREL} renamed PERI_POW
- net ~{BATT_PWR} renamed BATT_PWR
- new net IO33: U1.42 (GPIO33)
- new net IO34: U1.43 (GPIO34)
- new net IO35: U1.44 (GPIO35)
