File: Hardware/peripherals.kicad_sch (KiCad schematic)
At the start: 21 parts, among them J13 microSD, SW1 BOOT, SW2 RESET, SW3 USER

Commit message: Update v01 from checklist. Added measures.
Parts:
- renumbered J13 to J14, R24 to R26, R25 to R27, R26 to R28, R27 to R29, R28 to R30, R29 to R31, R30 to R32, TP12 to TP10, TP13 to TP11, TP11 to TP9

Commit message: v01 post design review changes. Panelize/CAM.
Remove F3.
Added switched power for qwiic, rgb, sd.
Update USB diode for prod friendly package.
Added debounce cap on User button.
Swap user and boot buttons.
Make F2 a smaller package.
Renumber GPIO and use contiguous numbers for PIO purposes.
Swap inputs on Ideal diodes for battery powered current purposes.
Move USB termination resistors closer to MCU.
Fixed A0-A5 ordering.
Update silks.
Add mask to middle of SMD GPIOs.
Parts:
- added C36: 0.1uF, SparkFun-Capacitor:C_0402_1005Metric, symbol SparkFun-Capacitor:0.1uF_0402_16V_10%
- added R33: 10k, SparkFun-Resistor:R_0402_1005Metric, symbol SparkFun-Resistor:10k_0402
- renumbered C32 to C34, C33 to C35, R26 to R28, R27 to R29, R28 to R30, R29 to R31, R30 to R32, R31 to R34, R32 to R35
Connections:
- net 3.3V: no longer C34.1, C35.1, D4.4 (VDD), J14.4 (VDD)
- net GND: now also C36.2
- net ~{SD_DET}: now also R33.1
- net ~{USER_BTN}: now also C36.1
- new net 3.3V_P: C34.1, C35.1, D4.4 (VDD), J14.4 (VDD), R33.2
Other:
- moved on the sheet: C35, J14
